Commit message: Modified to have base link

File: racecar_utils/urdf/av21.urdf (robot description, URDF)
Before this commit: robot AV21, 19 links, 18 joints
Links:
- removed link camera_front_1
- removed link camera_front_2
- removed link center_of_gravity
- removed link rear_axle_middle
- added link base_link
- added link camera_front_left_center
- added link camera_front_right_center
- added link cg
Joints:
- removed joint camera_front_1_joint
- removed joint camera_front_2_joint
- added joint camera_front_left_center_joint: type fixed, parent base_link, child camera_front_left_center, origin xyz=2.235 0.121 0.422
- added joint camera_front_right_center_joint: type fixed, parent base_link, child camera_front_right_center, origin xyz=2.235 -0.121 0.422
- joint camera_front_left_joint: parent rear_axle_middle -> base_link
- joint camera_front_right_joint: parent rear_axle_middle -> base_link
- joint camera_rear_left_joint: parent rear_axle_middle -> base_link
- joint camera_rear_right_joint: parent rear_axle_middle -> base_link
- joint luminar_front_joint: parent rear_axle_middle -> base_link
- joint luminar_left_joint: parent rear_axle_middle -> base_link
- joint luminar_right_joint: parent rear_axle_middle -> base_link
- joint radar_front_joint: parent rear_axle_middle -> base_link
- joint radar_port_joint: parent rear_axle_middle -> base_link
- joint radar_rear_joint: parent rear_axle_middle -> base_link
- joint radar_starboard_joint: parent rear_axle_middle -> base_link

Commit message: Still Debugging

File: racecar_utils/urdf/av21.urdf (robot description, URDF)
Before this commit: robot AV21, 19 links, 18 joints
Links:
- removed link imu_link
- added link base_footprint
- added link front_axle_middle
- added link imu_bottom
- added link imu_top
- added link imu_vectornav
- added link model; visual mesh filename=package://race_metadata/urdf/iac_car/visual/il15_body.stl scale=0.01 0.01 0.01
- added link nav_base
- added link rear_axle_middle
- added link tyre_fl; visual mesh filename=package://race_metadata/urdf/iac_car/visual/il15_tyre_fl.stl scale=0.01 0.01 0.01
- added link tyre_fr; visual mesh filename=package://race_metadata/urdf/iac_car/visual/il15_tyre_fr.stl scale=0.01 0.01 0.01
- added link tyre_rl; visual mesh filename=package://race_metadata/urdf/iac_car/visual/il15_tyre_rl.stl scale=0.01 0.01 0.01
- added link tyre_rr; visual mesh filename=package://race_metadata/urdf/iac_car/visual/il15_tyre_rr.stl scale=0.01 0.01 0.01
- added link vectornav
- added link vimba_front_left
- added link vimba_front_left_center
- added link vimba_front_right
- added link vimba_front_right_center
- added link vimba_rear_left
- added link vimba_rear_right
- link rear_axle_middle_ground: geometry 
Joints:
- removed joint imu_joint
- added joint base_footprint_joint: type fixed, parent base_link, child base_footprint, origin xyz=0 0 -0.09525
- added joint cg_joint: type fixed, parent base_link, child cg, origin xyz=1.248 0.0 0.077
- added joint fl_tyre_joint: type fixed, parent front_axle_middle, child tyre_fl, origin xyz=0.0 0.819 0.0 rpy=0 0 1.5708
- added joint fr_tyre_joint: type fixed, parent front_axle_middle, child tyre_fr, origin xyz=0.0 -0.819 0.0 rpy=0 0 1.5708
- added joint imu_bottom_joint: type fixed, parent base_link, child imu_bottom, origin xyz=1.605 -0.075 -0.074
- added joint imu_top_joint: type fixed, parent base_link, child imu_top, origin xyz=1.605 0.075 -0.074
- added joint imu_vectornav_joint: type fixed, parent base_link, child imu_vectornav, origin xyz=1.765 0.0 0.035
- added joint model_joint: type fixed, parent base_link, child model, origin xyz=1.725 0.0 -0.31 rpy=1.5708 0.0 1.5708
- added joint nav_base_joint: type fixed, parent cg, child nav_base, origin xyz=0 0 0
- added joint rl_tyre_joint: type fixed, parent rear_axle_middle, child tyre_rl, origin xyz=0.0 0.762 0.0 rpy=0 0 1.5708
- added joint rr_tyre_joint: type fixed, parent rear_axle_middle, child tyre_rr, origin xyz=0.0 -0.762 0.0 rpy=0 0 1.5708
- added joint vectornav_joint: type fixed, parent base_link, child vectornav, origin xyz=1.765 0.0 0.035
- added joint vimba_front_left_center_joint: type fixed, parent camera_front_left_center, child vimba_front_left_center, origin xyz=0 0 0 rpy=-1.5708 0 -1.5708
- added joint vimba_front_left_joint: type fixed, parent camera_front_left, child vimba_front_left, origin xyz=0 0 0 rpy=-1.5708 0 -1.5708
- added joint vimba_front_right_center_joint: type fixed, parent camera_front_right_center, child vimba_front_right_center, origin xyz=0 0 0 rpy=-1.5708 0 -1.5708
- added joint vimba_front_right_joint: type fixed, parent camera_front_right, child vimba_front_right, origin xyz=0 0 0 rpy=-1.5708 0 -1.5708
- added joint vimba_rear_left_joint: type fixed, parent camera_rear_left, child vimba_rear_left, origin xyz=0 0 0 rpy=-1.5708 0 -1.5708
- added joint vimba_rear_right_joint: type fixed, parent camera_rear_right, child vimba_rear_right, origin xyz=0 0 0 rpy=-1.5708 0 -1.5708
- added joint wheel_base: type fixed, parent base_link, child front_axle_middle, origin xyz=2.9718 0.0 0.0
- joint gps_bottom_joint: origin xyz=1.606 -0.05 -0.1428 -> xyz=1.605 -0.075 -0.074; parent rear_axle_middle -> base_link
- joint gps_top_joint: origin xyz=1.606 0.05 -0.1428 -> xyz=1.605 0.075 -0.074; parent rear_axle_middle -> base_link
- joint luminar_front_joint: origin xyz=2.342 0 0.448 -> xyz=2.242 0 0.448 rpy=0 0.0174533 0
- joint luminar_right_joint: origin xyz=1.549 -0.267 0.543 rpy=0 0 -2.0943951024 -> xyz=1.549 -0.267 0.543 rpy=-0.00872665 -0.0174533 -2.0943951024
- joint rear_axle_middle_ground_joint: child rear_axle_middle -> rear_axle_middle_ground; origin xyz=0 0 0.198 -> xyz=0.0 0.0 0.0; parent rear_axle_middle_ground -> base_footprint
- joint rear_axle_middle_joint: child center_of_gravity -> rear_axle_middle; origin xyz=1.3206 -0.030188 0.23598 -> xyz=0 0 0; parent rear_axle_middle -> base_link

Commit message: Should Work Perfectly now

File: racecar_utils/urdf/av21.urdf (robot description, URDF)
Before this commit: robot AV21, 19 links, 18 joints
Links:
- removed link camera_front_1
- removed link camera_front_2
- removed link center_of_gravity
- removed link imu_link
- added link base_footprint
- added link base_link
- added link camera_front_left_center
- added link camera_front_right_center
- added link cg
- added link front_axle_middle
- added link imu_bottom
- added link imu_top
- added link imu_vectornav
- added link model; visual mesh filename=package://race_metadata/urdf/iac_car/visual/il15_body.stl scale=0.01 0.01 0.01
- added link nav_base
- added link tyre_fl; visual mesh filename=package://race_metadata/urdf/iac_car/visual/il15_tyre_fl.stl scale=0.01 0.01 0.01
- added link tyre_fr; visual mesh filename=package://race_metadata/urdf/iac_car/visual/il15_tyre_fr.stl scale=0.01 0.01 0.01
- added link tyre_rl; visual mesh filename=package://race_metadata/urdf/iac_car/visual/il15_tyre_rl.stl scale=0.01 0.01 0.01
- added link tyre_rr; visual mesh filename=package://race_metadata/urdf/iac_car/visual/il15_tyre_rr.stl scale=0.01 0.01 0.01
- added link vectornav
- added link vimba_front_left
- added link vimba_front_left_center
- added link vimba_front_right
- added link vimba_front_right_center
- added link vimba_rear_left
- added link vimba_rear_right
- link rear_axle_middle_ground: geometry 
Joints:
- removed joint camera_front_1_joint
- removed joint camera_front_2_joint
- removed joint imu_joint
- added joint base_footprint_joint: type fixed, parent base_link, child base_footprint, origin xyz=0 0 -0.09525
- added joint camera_front_left_center_joint: type fixed, parent base_link, child camera_front_left_center, origin xyz=2.235 0.121 0.422
- added joint camera_front_right_center_joint: type fixed, parent base_link, child camera_front_right_center, origin xyz=2.235 -0.121 0.422
- added joint cg_joint: type fixed, parent base_link, child cg, origin xyz=1.248 0.0 0.077
- added joint fl_tyre_joint: type fixed, parent front_axle_middle, child tyre_fl, origin xyz=0.0 0.819 0.0 rpy=0 0 1.5708
- added joint fr_tyre_joint: type fixed, parent front_axle_middle, child tyre_fr, origin xyz=0.0 -0.819 0.0 rpy=0 0 1.5708
- added joint imu_bottom_joint: type fixed, parent base_link, child imu_bottom, origin xyz=1.605 -0.075 -0.074
- added joint imu_top_joint: type fixed, parent base_link, child imu_top, origin xyz=1.605 0.075 -0.074
- added joint imu_vectornav_joint: type fixed, parent base_link, child imu_vectornav, origin xyz=1.765 0.0 0.035
- added joint model_joint: type fixed, parent base_link, child model, origin xyz=1.725 0.0 -0.31 rpy=1.5708 0.0 1.5708
- added joint nav_base_joint: type fixed, parent cg, child nav_base, origin xyz=0 0 0
- added joint rl_tyre_joint: type fixed, parent rear_axle_middle, child tyre_rl, origin xyz=0.0 0.762 0.0 rpy=0 0 1.5708
- added joint rr_tyre_joint: type fixed, parent rear_axle_middle, child tyre_rr, origin xyz=0.0 -0.762 0.0 rpy=0 0 1.5708
- added joint vectornav_joint: type fixed, parent base_link, child vectornav, origin xyz=1.765 0.0 0.035
- added joint vimba_front_left_center_joint: type fixed, parent camera_front_left_center, child vimba_front_left_center, origin xyz=0 0 0 rpy=-1.5708 0 -1.5708
- added joint vimba_front_left_joint: type fixed, parent camera_front_left, child vimba_front_left, origin xyz=0 0 0 rpy=-1.5708 0 -1.5708
- added joint vimba_front_right_center_joint: type fixed, parent camera_front_right_center, child vimba_front_right_center, origin xyz=0 0 0 rpy=-1.5708 0 -1.5708
- added joint vimba_front_right_joint: type fixed, parent camera_front_right, child vimba_front_right, origin xyz=0 0 0 rpy=-1.5708 0 -1.5708
- added joint vimba_rear_left_joint: type fixed, parent camera_rear_left, child vimba_rear_left, origin xyz=0 0 0 rpy=-1.5708 0 -1.5708
- added joint vimba_rear_right_joint: type fixed, parent camera_rear_right, child vimba_rear_right, origin xyz=0 0 0 rpy=-1.5708 0 -1.5708
- added joint wheel_base: type fixed, parent base_link, child front_axle_middle, origin xyz=2.9718 0.0 0.0
- joint camera_front_left_joint: parent rear_axle_middle -> base_link
- joint camera_front_right_joint: parent rear_axle_middle -> base_link
- joint camera_rear_left_joint: parent rear_axle_middle -> base_link
- joint camera_rear_right_joint: parent rear_axle_middle -> base_link
- joint gps_bottom_joint: origin xyz=1.606 -0.05 -0.1428 -> xyz=1.605 -0.075 -0.074; parent rear_axle_middle -> base_link
- joint gps_top_joint: origin xyz=1.606 0.05 -0.1428 -> xyz=1.605 0.075 -0.074; parent rear_axle_middle -> base_link
- joint luminar_front_joint: origin xyz=2.342 0 0.448 -> xyz=2.242 0 0.448 rpy=0 0.0174533 0; parent rear_axle_middle -> base_link
- joint luminar_left_joint: parent rear_axle_middle -> base_link
- joint luminar_right_joint: origin xyz=1.549 -0.267 0.543 rpy=0 0 -2.0943951024 -> xyz=1.549 -0.267 0.543 rpy=-0.00872665 -0.0174533 -2.0943951024; parent rear_axle_middle -> base_link
- joint radar_front_joint: parent rear_axle_middle -> base_link
- joint radar_port_joint: parent rear_axle_middle -> base_link
- joint radar_rear_joint: parent rear_axle_middle -> base_link
- joint radar_starboard_joint: parent rear_axle_middle -> base_link
- joint rear_axle_middle_ground_joint: child rear_axle_middle -> base_link; origin xyz=0 0 0.198 -> xyz=0.0 0.0 -0.09525
- joint rear_axle_middle_joint: child center_of_gravity -> rear_axle_middle; origin xyz=1.3206 -0.030188 0.23598 -> xyz=0 0 0; parent rear_axle_middle -> base_link
